File: temp/temp.kicad_sch (KiCad schematic)
At the start: 22 parts, among them J1 USB_C_Receptacle_USB2.0_14P, SW1 BOOTSEL, SW2 RST, U1 STM32F103C8Tx, U2 SRV05-4, U3 AMS1117-3.3

Commit message: day 4
Parts:
- added Brd1: SSD1306, SSD1306:128x64OLED, symbol SSD1306-128x64_OLED:SSD1306
- added C1, C2, C4: 20pF, Capacitor_SMD:C_0201_0603Metric, symbol Device:C
- added C3: 15pF, Capacitor_SMD:C_0201_0603Metric, symbol Device:C
- added J2: MLX90614, Connector_PinHeader_2.54mm:PinHeader_1x04_P2.54mm_Vertical, symbol Connector:Conn_01x04_Pin
- added R2, R3: 1M, Resistor_SMD:R_0402_1005Metric, symbol Device:R
- added R5, R6: 20R, Resistor_SMD:R_0402_1005Metric, symbol Device:R
- added Y1: 8Mhz, Crystal:Crystal_SMD_3225-4Pin_3.2x2.5mm, symbol Device:Crystal_GND24
- added Y3: Crystal, Crystal:Crystal_SMD_3215-2Pin_3.2x1.5mm, symbol Device:Crystal
- C10: renamed from C8; footprint (none) -> Capacitor_SMD:C_0201_0603Metric
- C11: renamed from C9; footprint (none) -> Capacitor_SMD:C_0201_0603Metric
- C12: renamed from C2; footprint (none) -> Capacitor_SMD:C_0201_0603Metric
- C13: renamed from C1; footprint (none) -> Capacitor_SMD:C_0201_0603Metric
- C5: renamed from C3; footprint (none) -> Capacitor_SMD:C_0201_0603Metric
- C6: renamed from C4; footprint (none) -> Capacitor_SMD:C_0201_0603Metric
- C7: renamed from C5; footprint (none) -> Capacitor_SMD:C_0201_0603Metric
- C8: renamed from C6; footprint (none) -> Capacitor_SMD:C_0201_0603Metric
- C9: renamed from C7; footprint (none) -> Capacitor_SMD:C_0201_0603Metric
- D1: footprint (none) -> LED_SMD:LED_0603_1608Metric
- FB1: footprint Inductor_SMD:L_12x12mm_H8mm -> Inductor_SMD:L_0603_1608Metric_Pad1.05x0.95mm_HandSolder
- J1: footprint (none) -> Connector_USB:USB_C_Receptacle_GCT_USB4105-xx-A_16P_TopMnt_Horizontal
- R1: renamed from R3; footprint (none) -> Resistor_SMD:R_0402_1005Metric
- R4: footprint (none) -> Resistor_SMD:R_0402_1005Metric
- R7: renamed from R2; footprint (none) -> Resistor_SMD:R_0402_1005Metric
- R8: renamed from R1; footprint (none) -> Resistor_SMD:R_0402_1005Metric
- R9: renamed from 5.1K; value R -> 5.1k; footprint (none) -> Resistor_SMD:R_0402_1005Metric
- SW1, SW2: footprint (none) -> TS-1088-AR02016:SW_TS-1088-AR02016
- renumbered U3 to U2, U2 to U3
Connections:
- net +3V3: now also Brd1.2 (VCC), J2.1 (Pin_1)
- net D+: now also R6.1; no longer U1.33 (PA12)
- net D-: now also R5.2; no longer U1.32 (PA11)
- net GND: now also Brd1.1 (GND), C1.2, C2.2, C3.2, C4.1, J2.2 (Pin_2), Y1.1, Y1.3
- net PB0: now reaches U1.18 (PB0)
- net PB1: now reaches U1.19 (PB1)
- net PB2: now reaches U1.20 (PB2)
- net SCL: now reaches U1.21 (PB10)
- net SCL: now also Brd1.3 (SCL), J2.3 (Pin_3)
- net SDA: now reaches U1.22 (PB11)
- net SDA: now also Brd1.4 (SDA), J2.4 (Pin_4)
- net PC14: now reaches U1.3 (PC14)
- net PC14: now also C3.1, R3.1, Y3.2
- net PB3: now reaches U1.39 (PB3)
- net PC15: now reaches U1.4 (PC15)
- net PC15: now also C4.2, R3.2, Y3.1
- net PB4: now reaches U1.40 (PB4)
- net PB5: now reaches U1.41 (PB5)
- net OSC_IN: now reaches U1.5 (PD0)
- net OSC_IN: now also C1.1, R2.1, Y1.2
- net OSC_OUT: now reaches U1.6 (PD1)
- net OSC_OUT: now also C2.1, R2.2, Y1.4
- new net: R5.1, U1.32 (PA11)
- new net: R6.2, U1.33 (PA12)
Other:
- moved on the sheet: R7

Commit message: pcb fully done now time for case
Parts:
- removed Brd1: SSD1306, SSD1306:128x64OLED, symbol SSD1306-128x64_OLED:SSD1306
- removed R2: 1M, Resistor_SMD:R_0402_1005Metric, symbol Device:R
- added D2, D3: LED, LED_SMD:LED_0603_1608Metric, symbol Device:LED
- added J3: OLED, Connector_PinHeader_2.54mm:PinHeader_1x04_P2.54mm_Vertical, symbol Connector:Conn_01x04_Pin
- added J5: Conn_02x10_Counter_Clockwise, Connector_PinSocket_2.54mm:PinSocket_2x10_P2.54mm_Vertical, symbol Connector_Generic:Conn_02x10_Counter_Clockwise
- added R10, R11: 330, Resistor_SMD:R_0402_1005Metric, symbol Device:R
- C1, C10, C11, C2, C4, C6, C7, C8, C9: footprint Capacitor_SMD:C_0201_0603Metric -> Capacitor_SMD:C_0402_1005Metric
- C12, C13, C5: footprint Capacitor_SMD:C_0201_0603Metric -> Capacitor_SMD:C_0603_1608Metric
- C3: value 15pF -> 20pF; footprint Capacitor_SMD:C_0201_0603Metric -> Capacitor_SMD:C_0402_1005Metric
- R3: value 1M -> 0
Connections:
- net +3V3: now also D3.2 (A), J3.1 (Pin_1), J5.11 (Pin_11)
- net +5V: now also U3.5 (VP), D2.2 (A)
- net D+: now also U3.4 (IO3); no longer U3.6 (IO4)
- net D-: now also U3.6 (IO4); no longer U3.4 (IO3)
- net GND: now also U3.2 (VN), J3.2 (Pin_2), J5.10 (Pin_10), R10.2, R11.2
- net PC14: no longer R3.1
- net PC15: no longer C4.2, Y3.1
- net SCL: now also J3.3 (Pin_3), J5.9 (Pin_9)
- net SDA: now also J3.4 (Pin_4), J5.12 (Pin_12)
- net A1: now reaches U1.13 (PA3)
- net A1: now also J5.19 (Pin_19)
- net A2: now reaches U1.14 (PA4)
- net A2: now also J5.18 (Pin_18)
- net A3: now reaches U1.15 (PA5)
- net A3: now also J5.17 (Pin_17)
- net A4: now reaches U1.16 (PA6)
- net A4: now also J5.16 (Pin_16)
- net A5: now reaches U1.17 (PA7)
- net A5: now also J5.15 (Pin_15)
- net Di-: now reaches R5.1, U1.32 (PA11)
- net Di+: now reaches R6.2, U1.33 (PA12)
- net B9: now reaches U1.37 (PA14)
- net B9: now also J5.1 (Pin_1)
- net B8: now reaches U1.38 (PA15)
- net B8: now also J5.2 (Pin_2)
- net B4: now reaches U1.42 (PB6)
- net B4: now also J5.6 (Pin_6)
- net B3: now reaches U1.43 (PB7)
- net B3: now also J5.7 (Pin_7)
- net B2: now reaches U1.45 (PB8)
- net B2: now also J5.8 (Pin_8)
- net B1: now reaches U1.46 (PB9)
- net B1: now also J5.20 (Pin_20)
- net DU+: now reaches J1.A6 (D+), J1.B6 (D+), U3.3 (IO2)
- net DU-: now reaches J1.A7 (D-), J1.B7 (D-), U3.1 (IO1)
- net PB0 renamed A6
- net A6: now also J5.14 (Pin_14)
- net PB1 renamed A7
- net A7: now also J5.13 (Pin_13)
- net PB2: no longer names the net of U1.20 (PB2)
- net PB3 renamed B7
- net B7: now also J5.3 (Pin_3)
- net PB4 renamed B6
- net B6: now also J5.4 (Pin_4)
- net PB5 renamed B5
- net B5: now also J5.5 (Pin_5)
- new net: D3.1 (K), R11.1
- new net: D2.1 (K), R10.1
- new net: C4.2, R3.1, Y3.1
Other:
- moved on the sheet: R3
