File: temp/temp.kicad_pcb (KiCad board)
At the start: 2 copper layers, 36 x 40 mm, 34 parts, among them J1 USB_C_Receptacle_USB2.0_14P, J2 MLX90614, SW1 BOOTSEL, SW2 RST, U1 STM32F103C8Tx, U2 AMS1117-3.3, U3 SRV05-4, Y1 8Mhz, Y3 Crystal

Commit message: pcb fully done now time for case
Parts:
- removed Brd1: SSD1306, SSD1306:128x64OLED
- removed R2: 1M, Resistor_SMD:R_0402_1005Metric
- added D2: LED, LED_SMD:LED_0603_1608Metric, F.Cu at (207.8, 103.5)
- added D3: LED, LED_SMD:LED_0603_1608Metric, F.Cu at (214.8, 114.0)
- added J3: OLED, Connector_PinHeader_2.54mm:PinHeader_1x04_P2.54mm_Vertical, F.Cu at (231.0, 116.6)
- added J5: Conn_02x10_Counter_Clockwise, Connector_PinSocket_2.54mm:PinSocket_2x10_P2.54mm_Vertical, F.Cu at (203.6, 134.7)
- added R10: 330, Resistor_SMD:R_0402_1005Metric, F.Cu at (206.2, 105.5)
- added R11: 330, Resistor_SMD:R_0402_1005Metric, F.Cu at (213.5, 115.2)
- C1, C10, C11, C2, C4, C6, C7, C8, C9: footprint Capacitor_SMD:C_0201_0603Metric -> Capacitor_SMD:C_0402_1005Metric
- C12, C13, C5: footprint Capacitor_SMD:C_0201_0603Metric -> Capacitor_SMD:C_0603_1608Metric
- C3: value 15pF -> 20pF; footprint Capacitor_SMD:C_0201_0603Metric -> Capacitor_SMD:C_0402_1005Metric
- R3: value 1M -> 0
- moved J2 106.0 mm to (227.0, 116.6), turned to 180 degrees
- moved SW2 105.4 mm to (227.5, 103.2)
- moved R3 104.4 mm to (224.8, 126.0), turned to 180 degrees
- moved C3 103.9 mm to (229.0, 128.5), turned to 90 degrees
- moved C4 100.9 mm to (229.0, 126.0), turned to 90 degrees
- moved C2 100.6 mm to (229.1, 121.6), turned to -90 degrees
- moved C1 100.0 mm to (224.0, 124.2), turned to 180 degrees
- moved U2 97.4 mm to (207.8, 114.5), turned to -90 degrees
- moved C6 94.3 mm to (221.5, 121.5)
- moved Y1 94.2 mm to (226.9, 122.9), turned to -90 degrees
- moved R4 93.7 mm to (218.8, 115.5)
- moved C11 93.6 mm to (217.8, 129.0), turned to -90 degrees
- moved C5 93.4 mm to (226.5, 119.2), turned to 180 degrees
- moved C9 92.8 mm to (220.8, 126.0), turned to -90 degrees
- moved Y3 89.6 mm to (226.9, 127.2), turned to 90 degrees
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Connections:
- net Net-(U1-PA11) renamed /Di-
- net Net-(U1-PA12) renamed /Di+
- net Net-(U3-IO1) renamed /DU-
- net Net-(U3-IO2) renamed /DU+
- C4 pad 2: /PC15 -> Net-(C4-Pad2)
- R3 pad 1: /PC14 -> Net-(C4-Pad2)
- U1 pad 13: unconnected-(U1-PA3-Pad13) -> /A1
- U1 pad 14: unconnected-(U1-PA4-Pad14) -> /A2
- U1 pad 15: unconnected-(U1-PA5-Pad15) -> /A3
- U1 pad 16: unconnected-(U1-PA6-Pad16) -> /A4
- U1 pad 17: unconnected-(U1-PA7-Pad17) -> /A5
- U1 pad 18: /PB0 -> /A6
- U1 pad 19: /PB1 -> /A7
- U1 pad 20: /PB2 -> unconnected-(U1-PB2-Pad20)
- U1 pad 37: unconnected-(U1-PA14-Pad37) -> /B9
- U1 pad 38: unconnected-(U1-PA15-Pad38) -> /B8
- U1 pad 39: /PB3 -> /B7
- U1 pad 40: /PB4 -> /B6
- U1 pad 41: /PB5 -> /B5
- U1 pad 42: unconnected-(U1-PB6-Pad42) -> /B4
- U1 pad 43: unconnected-(U1-PB7-Pad43) -> /B3
- U1 pad 45: unconnected-(U1-PB8-Pad45) -> /B2
- U1 pad 46: unconnected-(U1-PB9-Pad46) -> /B1
- U3 pad 2: unconnected-(U3-VN-Pad2) -> GND
- U3 pad 4: /D- -> /D+
- U3 pad 5: unconnected-(U3-VP-Pad5) -> +5V
- U3 pad 6: /D+ -> /D-
- Y3 pad 1: /PC15 -> Net-(C4-Pad2)
Routing:
- net GND: track 0.00 -> 101.7 mm, vias 0 -> 27
- net +3V3: track 0.00 -> 89.5 mm, vias 0 -> 13
- net /SDA: track 0.00 -> 44.8 mm, vias 0 -> 2
- net /SCL: track 0.00 -> 40.1 mm, vias 0 -> 1
- net +5V: track 0.00 -> 38.6 mm, vias 0 -> 4
- net Net-(U1-BOOT0): track 0.00 -> 37.1 mm, vias 0 -> 4
- net /B1: track 0.00 -> 28.0 mm, vias 0 -> 1
- net Net-(U1-NRST): track 0.00 -> 28.0 mm, vias 0 -> 4
- net /A7: track 0.00 -> 25.4 mm, vias 0 -> 1
- net Net-(J1-SHIELD): track 0.00 -> 24.7 mm, vias 0 -> 1
- net /A6: track 0.00 -> 24.5 mm, vias 0 -> 1
- net /A2: track 0.00 -> 23.9 mm, vias 0 -> 1
- net /A4: track 0.00 -> 22.9 mm, vias 0 -> 1
- net /A3: track 0.00 -> 21.3 mm, vias 0 -> 1
- net /A5: track 0.00 -> 21.0 mm, vias 0 -> 1
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- added copper zone on F.Cu, net +3V3
- added copper zone on B.Cu, net GND

Commit message: f
Parts:
- added REF**: MountingHole_2.2mm_M2_DIN965_Pad_TopBottom, MountingHole:MountingHole_2.2mm_M2_DIN965_Pad_TopBottom, F.Cu at (200.0, 130.0)
- moved C3 4.88 mm to (224.2, 127.6), turned to 180 degrees
- moved R3 1.00 mm to (224.0, 125.4)
- moved Y3 0.30 mm to (226.6, 127.2)
Routing:
- net /PC14: track 11.7 -> 9.11 mm
- net +3V3: track 89.5 -> 91.6 mm
- net /PC15: track 5.96 -> 4.91 mm
- net Net-(C4-Pad2): track 3.89 -> 4.90 mm
- net Net-(U1-BOOT0): track 37.1 -> 36.5 mm
